File: hw/xmas_ornament_2019.brd (EAGLE design)
At the start: 63.5 x 88.9 mm, 36 parts, among them J1 ARM_SWD_10_TAG, U1 TLV75533PDBVR, U2 ATSAMD21G18A-MUT, U3 PRTR5V0U2X, X1 FC-135 32.7680KA-A5

Commit message: Current progress.
Parts:
- moved R3 32.1 mm to (24.4, 25.3), turned to 180 degrees
- moved R2 0.90 mm to (28.2, 27.6)
Connections:
- new net D1: D1.A, R1.4
- new net D10: D10.A
- new net D2: D2.A
- new net D3: D3.A
- new net D4: D4.A
- new net D5: D5.A
- new net D6: D6.A
- new net D7: D7.A
- new net D8: D8.A
- new net D9: D9.A
- new net N$10: R3.5, U2.24
- new net N$11: R3.6, U2.23
Routing:
- net D1: track 0.00 -> 31.1 mm
- net N$10: track 0.00 -> 9.28 mm
- net N$11: track 0.00 -> 8.30 mm
- net GND: track 79.5 -> 72.0 mm

Commit message: Added artwork
Parts:
- moved D1 1.26 mm to (6.99, 20.6), turned to 35 degrees
- moved D4 0.13 mm to (20.6, 30.0)
Connections:
- net D10: now also R2.1
- net D2: now also R1.2
- net D3: now also R1.3
- net D4: now also R1.1
- net D5: now also R3.4
- net D6: now also R3.3
- net D7: now also R2.4
- net D8: now also R2.3
- net D9: now also R2.2
Routing:
- net D6: track 0.00 -> 61.5 mm
- net D2: track 0.00 -> 51.2 mm
- net D5: track 0.00 -> 49.7 mm
- net D7: track 0.00 -> 49.7 mm
- net D8: track 0.00 -> 41.6 mm
- net D3: track 0.00 -> 39.0 mm
- net D10: track 0.00 -> 36.6 mm
- net D9: track 0.00 -> 31.0 mm
- net D4: track 0.00 -> 13.3 mm
- net GND: track 72.0 -> 74.1 mm, vias 30 -> 31
- net D1: track 31.1 -> 30.2 mm
- net VCC: track 90.1 -> 90.8 mm

Commit message: Rev A.
Parts:
- removed TP1: TPTP-PTH0.02, jetperch:TP-PTH0.02
- J2: value (none) -> BU2450-SM-JJ-GTR
- P1: value (none) -> PCB_connector
- SW1: value (none) -> JS203011SCQN
- SW2: value (none) -> PTS645SM43SMTR92 LFS
- renumbered B1 to J2, B2 to SW2, S1 to SW1
Connections:
- new net BUTTON: SW2.1, SW2.2, U2.7
- net !BATTERY: now also U2.9
- net VREFA: no longer TP1.1
Routing:
- net !BATTERY: track 0.00 -> 31.6 mm, vias 0 -> 2
- net BUTTON: track 0.00 -> 28.0 mm
- net GND: track 74.1 -> 72.7 mm
- net VREFA: track 3.07 -> 1.92 mm
- net VUSB_3V3: track 14.6 -> 13.7 mm
- net VDD_ANA: track 11.0 -> 10.3 mm
- net D2: track 51.2 -> 50.7 mm
- net D1: track 30.2 -> 29.7 mm
- net D3: track 39.0 -> 38.5 mm
- net VCC: track 90.8 -> 91.2 mm, vias 7 -> 8
Other:
- board size 63.5 x 88.9 mm -> 63.5 x 91.4 mm
- board text added: "From the Libertys Matt, Shelly, Eleanor & Nicholas"
