File: hw/xmas_ornament_2019.sch (EAGLE design)
At the start: 36 parts, among them J1 ARM_SWD_10_TAG, U1 TLV75533PDBVR, U2 ATSAMD21G18A-MUT, U3 PRTR5V0U2X, X1 FC-135 32.7680KA-A5

Commit message: Current progress.
Connections:
- new net D1: D1.A, R1.4A
- new net D10: D10.A
- new net D2: D2.A
- new net D3: D3.A
- new net D4: D4.A
- new net D5: D5.A
- new net D6: D6.A
- new net D7: D7.A
- new net D8: D8.A
- new net D9: D9.A
- new net N$10: R3.4B, U2.PA15/D5
- new net N$11: R3.3B, U2.PA14/D2
Other:
- moved on the sheet: D1, D10, D2, D3, D4, D5, D6, D8, D9, R2, R3

Commit message: Added artwork
Connections:
- net D10: now also R2.1A
- net D2: now also R1.2A
- net D3: now also R1.3A
- net D4: now also R1.1A
- net D5: now also R3.4A
- net D6: now also R3.3A
- net D7: now also R2.4A
- net D8: now also R2.3A
- net D9: now also R2.2A
Changed lines of the file:
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@@
 <?xml version="1.0" encoding="utf-8"?>
 <!DOCTYPE eagle SYSTEM "eagle.dtd">
-<eagle version="9.5.1">
+<eagle version="9.5.2">
 <drawing>
 <settings>
@@
 <label x="58.42" y="175.26" size="1.778" layer="95" rot="R90"/>
 </segment>
+<segment>
+<pinref part="R1" gate="G$1" pin="2A"/>
+<wire x1="365.76" y1="116.84" x2="378.46" y2="116.84" width="0.1524" layer="91"/>
+<label x="378.46" y="116.84" size="1.778" layer="95"/>
+</segment>
 </net>
 <net name="D3" class="0">
@@
 <label x="66.04" y="175.26" size="1.778" layer="95" rot="R90"/>
 </segment>
+<segment>
+<pinref part="R1" gate="G$1" pin="3A"/>
+<wire x1="365.76" y1="119.38" x2="378.46" y2="119.38" width="0.1524" layer="91"/>
+<label x="378.46" y="119.38" size="1.778" layer="95"/>
+</segment>
 </net>
 <net name="D4" class="0">
@@
 <label x="73.66" y="175.26" size="1.778" layer="95" rot="R90"/>
 </segment>
+<segment>
+<pinref part="R1" gate="G$1" pin="1A"/>
+<wire x1="365.76" y1="114.3" x2="378.46" y2="114.3" width="0.1524" layer="91"/>
+<label x="378.46" y="114.3" size="1.778" layer="95"/>
+</segment>
 </net>
 <net name="D5" class="0">
@@
 <label x="81.28" y="175.26" size="1.778" layer="95" rot="R90"/>
 </segment>
+<segment>
+<pinref part="R3" gate="G$1" pin="4A"/>
+<wire x1="299.72" y1="60.96" x2="299.72" y2="55.88" width="0.1524" layer="91"/>
+<wire x1="299.72" y1="55.88" x2="309.88" y2="55.88" width="0.1524" layer="91"/>
+<label x="309.88" y="55.88" size="1.778" layer="95"/>
+</segment>
 </net>
 <net name="D6" class="0">
@@
 <label x="88.9" y="175.26" size="1.778" layer="95" rot="R90"/>
 </segment>
+<segment>
+<pinref part="R3" gate="G$1" pin="3A"/>
+<wire x1="297.18" y1="60.96" x2="297.18" y2="53.34" width="0.1524" layer="91"/>
+<wire x1="297.18" y1="53.34" x2="309.88" y2="53.34" width="0.1524" layer="91"/>
+<label x="309.88" y="53.34" size="1.778" layer="95"/>
+</segment>
 </net>
 <net name="D7" class="0">
@@
 <label x="96.52" y="175.26" size="1.778" layer="95" rot="R90"/>
 </segment>
+<segment>
+<pinref part="R2" gate="G$1" pin="4A"/>
+<wire x1="261.62" y1="60.96" x2="261.62" y2="58.42" width="0.1524" layer="91"/>
+<wire x1="261.62" y1="58.42" x2="266.7" y2="58.42" width="0.1524" layer="91"/>
+<label x="266.7" y="58.42" size="1.778" layer="95"/>
+</segment>
 </net>
 <net name="D8" class="0">
@@
 <label x="104.14" y="175.26" size="1.778" layer="95" rot="R90"/>
 </segment>
+<segment>
+<pinref part="R2" gate="G$1" pin="3A"/>
+<wire x1="259.08" y1="60.96" x2="259.08" y2="55.88" width="0.1524" layer="91"/>
+<wire x1="259.08" y1="55.88" x2="266.7" y2="55.88" width="0.1524" layer="91"/>
+<label x="266.7" y="55.88" size="1.778" layer="95"/>
+</segment>
 </net>
 <net name="D9" class="0">
@@
 <label x="111.76" y="175.26" size="1.778" layer="95" rot="R90"/>
 </segment>
+<segment>
+<pinref part="R2" gate="G$1" pin="2A"/>
+<wire x1="256.54" y1="60.96" x2="256.54" y2="53.34" width="0.1524" layer="91"/>
+<wire x1="256.54" y1="53.34" x2="266.7" y2="53.34" width="0.1524" layer="91"/>
+<label x="266.7" y="53.34" size="1.778" layer="95"/>
+</segment>
 </net>
 <net name="D10" class="0">
@@
 <label x="119.38" y="175.26" size="1.778" layer="95" rot="R90"/>
 </segment>
-</net>
+<segment>
+<pinref part="R2" gate="G$1" pin="1A"/>
+<wire x1="254" y1="60.96" x2="254" y2="50.8" width="0.1524" layer="91"/>
+<wire x1="254" y1="50.8" x2="266.7" y2="50.8" width="0.1524" layer="91"/>
+<label x="266.7" y="50.8" size="1.778" layer="95"/>
+</segment>
+</net>

Commit message: Rev A.
Parts:
- removed TP1: TPTP-PTH0.02, jetperch:TPTP-PTH0.02
- J2: value (none) -> BU2450-SM-JJ-GTR; MPN (none) -> BU2450-SM-JJ-GTR; POPULATE (none) -> 1
- P1: value (none) -> PCB_connector; POPULATE (none) -> 0
- SW1: value (none) -> JS203011SCQN; MPN (none) -> JS203011SCQN; POPULATE (none) -> 1
- SW2: value (none) -> PTS645SM43SMTR92 LFS; MPN (none) -> PTS645SM43SMTR92 LFS; POPULATE (none) -> 1
- renumbered B1 to J2, B2 to SW2, S1 to SW1
Connections:
- new net BUTTON: SW2.P$1, U2.PB08/A1
- net !BATTERY: now also U2.PA04/A3
- net VREFA: no longer TP1.TP
Changed lines of the file:
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@@
 </part>
 <part name="PWR9" library="jetperch" deviceset="GND_EARTH" device=""/>
-<part name="TP1" library="jetperch" deviceset="TP" device="TP-PTH0.02"/>
-<part name="P1" library="jetperch" deviceset="USB-4-PCB" device="-A"/>
-<part name="S1" library="jetperch" deviceset="SWITCH-DP3T" device="_JS203011SCQN"/>
-<part name="B1" library="jetperch" deviceset="BATTERY" device="_BU2450SM-JJ-G"/>
+<part name="P1" library="jetperch" deviceset="USB-4-PCB" device="-A" value="PCB_connector">
+<attribute name="POPULATE" value="0"/>
+</part>
+<part name="SW1" library="jetperch" deviceset="SWITCH-DP3T" device="_JS203011SCQN" value="JS203011SCQN">
+<attribute name="MPN" value="JS203011SCQN"/>
+<attribute name="POPULATE" value="1"/>
+</part>
+<part name="J2" library="jetperch" deviceset="BATTERY" device="_BU2450SM-JJ-G" value="BU2450-SM-JJ-GTR">
+<attribute name="MPN" value="BU2450-SM-JJ-GTR"/>
+<attribute name="POPULATE" value="1"/>
+</part>
 <part name="PWR6" library="jetperch" deviceset="GND_EARTH" device=""/>
 <part name="D6" library="jetperch" deviceset="LED" device="0805_BREV" value="APT2012LSYCK/J3-PRV">
@@
 <attribute name="WATTAGE" value="0.062W"/>
 </part>
-<part name="B2" library="jetperch" deviceset="SWITCH-SPST-NO" device=""/>
+<part name="SW2" library="jetperch" deviceset="SWITCH-SPST-NO" device="" value="PTS645SM43SMTR92 LFS">
+<attribute name="MPN" value="PTS645SM43SMTR92 LFS"/>
+<attribute name="POPULATE" value="1"/>
+</part>
 <part name="PWR7" library="jetperch" deviceset="GND_EARTH" device=""/>
 <part name="PWR8" library="jetperch" deviceset="GND_EARTH" device=""/>
@@
 </instance>
 <instance part="PWR9" gate="G$1" x="213.36" y="96.52" smashed="yes"/>
-<instance part="TP1" gate="G$1" x="205.74" y="147.32" smashed="yes" rot="R180">
-<attribute name="NAME" x="203.2" y="147.32" size="1.27" layer="95" rot="R180" align="center-left"/>
-</instance>
 <instance part="P1" gate="G1" x="30.48" y="45.72" smashed="yes" rot="MR0">
 <attribute name="NAME" x="38.1" y="53.848" size="1.778" layer="95" rot="MR0"/>
 <attribute name="VALUE" x="29.464" y="38.1" size="1.778" layer="96" rot="MR0"/>
-</instance>
-<instance part="S1" gate="G$1" x="198.12" y="58.42" smashed="yes" rot="MR0">
+<attribute name="POPULATE" x="30.48" y="45.72" size="1.778" layer="96" rot="MR0" display="off"/>
+</instance>
+<instance part="SW1" gate="G$1" x="198.12" y="58.42" smashed="yes" rot="MR0">
 <attribute name="NAME" x="200.66" y="66.04" size="1.27" layer="95" rot="MR0"/>
-</instance>
-<instance part="B1" gate="G$1" x="142.24" y="73.66" smashed="yes"/>
+<attribute name="MPN" x="198.12" y="58.42" size="1.778" layer="96" rot="MR0" display="off"/>
+<attribute name="POPULATE" x="198.12" y="58.42" size="1.778" layer="96" rot="MR0" display="off"/>
+</instance>
+<instance part="J2" gate="G$1" x="142.24" y="73.66" smashed="yes">
+<attribute name="MPN" x="142.24" y="73.66" size="1.778" layer="96" display="off"/>
+<attribute name="POPULATE" x="142.24" y="73.66" size="1.778" layer="96" display="off"/>
+</instance>
 <instance part="PWR6" gate="G$1" x="142.24" y="60.96" smashed="yes"/>
 <instance part="D6" gate="G$1" x="88.9" y="167.64" smashed="yes">
@@
 <attribute name="VALUE" x="362.966" y="126.746" size="1.27" layer="95" rot="R180"/>
 </instance>
-<instance part="B2" gate="G$1" x="99.06" y="109.22" smashed="yes" rot="MR0">
+<instance part="SW2" gate="G$1" x="99.06" y="109.22" smashed="yes" rot="MR0">
 <attribute name="NAME" x="98.552" y="109.474" size="1.778" layer="95" rot="MR0"/>
+<attribute name="MPN" x="99.06" y="109.22" size="1.778" layer="96" rot="MR0" display="off"/>
+<attribute name="POPULATE" x="99.06" y="109.22" size="1.778" layer="96" rot="MR0" display="off"/>
 </instance>
 <instance part="PWR7" gate="G$1" x="187.96" y="43.18" smashed="yes"/>
@@
 </segment>
 <segment>
-<pinref part="B1" gate="G$1" pin="-"/>
+<pinref part="J2" gate="G$1" pin="-"/>
 <pinref part="PWR6" gate="G$1" pin="GND"/>
 <wire x1="142.24" y1="68.58" x2="142.24" y2="66.04" width="0.1524" layer="91"/>
-<pinref part="S1" gate="G$1" pin="A1"/>
+<pinref part="SW1" gate="G$1" pin="A1"/>
 <wire x1="142.24" y1="66.04" x2="142.24" y2="63.5" width="0.1524" layer="91"/>
 <wire x1="190.5" y1="66.04" x2="142.24" y2="66.04" width="0.1524" layer="91"/>
@@
 </segment>
 <segment>
-<pinref part="S1" gate="G$1" pin="B2"/>
+<pinref part="SW1" gate="G$1" pin="B2"/>
 <wire x1="190.5" y1="53.34" x2="187.96" y2="53.34" width="0.1524" layer="91"/>
 <pinref part="PWR7" gate="G$1" pin="GND"/>
 <wire x1="187.96" y1="53.34" x2="187.96" y2="45.72" width="0.1524" layer="91"/>
-<pinref part="S1" gate="G$1" pin="A2"/>
+<pinref part="SW1" gate="G$1" pin="A2"/>
 <wire x1="190.5" y1="63.5" x2="187.96" y2="63.5" width="0.1524" layer="91"/>
 <wire x1="187.96" y1="63.5" x2="187.96" y2="53.34" width="0.1524" layer="91"/>
@@
 </segment>
 <segment>
-<pinref part="B2" gate="G$1" pin="P$2"/>
+<pinref part="SW2" gate="G$1" pin="P$2"/>
 <wire x1="93.98" y1="109.22" x2="91.44" y2="109.22" width="0.1524" layer="91"/>
 <pinref part="PWR10" gate="G$1" pin="GND"/>
@@
 </segment>
 <segment>
-<pinref part="S1" gate="G$1" pin="B_COM"/>
+<pinref part="SW1" gate="G$1" pin="B_COM"/>
 <wire x1="203.2" y1="53.34" x2="205.74" y2="53.34" width="0.1524" layer="91"/>
 <label x="213.36" y="53.34" size="1.778" layer="95"/>
@@
 <wire x1="213.36" y1="147.32" x2="213.36" y2="111.76" width="0.1524" layer="91"/>
 <pinref part="C5" gate="A" pin="2"/>
-<pinref part="TP1" gate="G$1" pin="TP"/>
-<wire x1="213.36" y1="147.32" x2="210.82" y2="147.32" width="0.1524" layer="91"/>
-<junction x="213.36" y="147.32"/>
 <label x="218.44" y="147.32" size="1.27" layer="95"/>
 </segment>
@@
 <segment>
 <pinref part="U1" gate="G$1" pin="OUT"/>
-<pinref part="S1" gate="G$1" pin="B3"/>
+<pinref part="SW1" gate="G$1" pin="B3"/>
 <wire x1="172.72" y1="50.8" x2="182.88" y2="50.8" width="0.1524" layer="91"/>
 <wire x1="182.88" y1="50.8" x2="190.5" y2="50.8" width="0.1524" layer="91"/>
-<pinref part="S1" gate="G$1" pin="A3"/>
+<pinref part="SW1" gate="G$1" pin="A3"/>
 <wire x1="190.5" y1="60.96" x2="182.88" y2="60.96" width="0.1524" layer="91"/>
 <wire x1="182.88" y1="60.96" x2="182.88" y2="50.8" width="0.1524" layer="91"/>
@@
 <segment>
 <wire x1="177.8" y1="81.28" x2="142.24" y2="81.28" width="0.1524" layer="91"/>
-<pinref part="B1" gate="G$1" pin="+"/>
+<pinref part="J2" gate="G$1" pin="+"/>
 <wire x1="142.24" y1="81.28" x2="142.24" y2="78.74" width="0.1524" layer="91"/>
-<pinref part="S1" gate="G$1" pin="B1"/>
+<pinref part="SW1" gate="G$1" pin="B1"/>
 <wire x1="190.5" y1="55.88" x2="177.8" y2="55.88" width="0.1524" layer="91"/>
 <wire x1="177.8" y1="55.88" x2="177.8" y2="81.28" width="0.1524" layer="91"/>
@@
 <net name="!BATTERY" class="0">
 <segment>
-<pinref part="S1" gate="G$1" pin="A_COM"/>
-<wire x1="203.2" y1="63.5" x2="213.36" y2="63.5" width="0.1524" layer="91"/>
-<label x="213.36" y="63.5" size="1.778" layer="95"/>
+<pinref part="SW1" gate="G$1" pin="A_COM"/>
+<wire x1="203.2" y1="63.5" x2="218.44" y2="63.5" width="0.1524" layer="91"/>
+<label x="205.74" y="63.5" size="1.778" layer="95"/>
+<pinref part="U2" gate="G$1" pin="PA04/A3"/>
+<wire x1="226.06" y1="132.08" x2="218.44" y2="132.08" width="0.1524" layer="91"/>
+<wire x1="218.44" y1="132.08" x2="218.44" y2="63.5" width="0.1524" layer="91"/>
 </segment>
 </net>
@@
 </segment>
 </net>
+<net name="BUTTON" class="0">
+<segment>
+<pinref part="SW2" gate="G$1" pin="P$1"/>
+<label x="121.92" y="109.22" size="1.778" layer="95"/>
+<pinref part="U2" gate="G$1" pin="PB08/A1"/>
+<wire x1="226.06" y1="142.24" x2="170.18" y2="142.24" width="0.1524" layer="91"/>
+<wire x1="170.18" y1="142.24" x2="170.18" y2="109.22" width="0.1524" layer="91"/>
+<wire x1="170.18" y1="109.22" x2="109.22" y2="109.22" width="0.1524" layer="91"/>
+</segment>
+</net>
